Commit message: feat: completar fase 2 y activar fase 4

File: simulacion/simulacion_dron/urdf/dron.xacro (robot description, xacro)
@@ -45,5 +45,5 @@
         </collision>
         <inertial>
-            <mass value="1.0"/>
+            <mass value="${fisico_cuerpo_masa}"/>
             <inertia ixx="${fisico_cuerpo_matriz_inercia.split()[0]}" iyy="${fisico_cuerpo_matriz_inercia.split()[1]}" izz="${fisico_cuerpo_matriz_inercia.split()[2]}" ixy="${fisico_cuerpo_matriz_inercia.split()[3]}" ixz="${fisico_cuerpo_matriz_inercia.split()[4]}" iyz="${fisico_cuerpo_matriz_inercia.split()[5]}"/>
         </inertial>

File: simulacion/simulacion_dron/urdf/dron_plugins.xacro (robot description, xacro)
@@ -70,5 +70,5 @@
         </collision>
         <inertial>
-            <mass value="1.0"/>
+            <mass value="${fisico_cuerpo_masa}"/>
             <inertia ixx="${fisico_cuerpo_matriz_inercia.split()[0]}" iyy="${fisico_cuerpo_matriz_inercia.split()[1]}" izz="${fisico_cuerpo_matriz_inercia.split()[2]}" ixy="${fisico_cuerpo_matriz_inercia.split()[3]}" ixz="${fisico_cuerpo_matriz_inercia.split()[4]}" iyz="${fisico_cuerpo_matriz_inercia.split()[5]}"/>
         </inertial>
